File: v0.9/PERIPHERALS.kicad_sch (KiCad schematic)
At the start: 12 parts, among them SW1 SW_Push, SW2 SW_Push

Commit message: Add files via upload
status LEDs added
Parts:
- C12, C9: LCSC Part Number C1711 -> C49678
- renumbered R10 to R14, R11 to R15
Changed lines of the file:
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@@
       (effects (font (size 1.27 1.27)) hide)
     )
-    (property "LCSC Part Number" "C1711" (id 5) (at 81.28 125.73 0)
+    (property "LCSC Part Number" "C49678" (id 5) (at 81.28 125.73 0)
       (effects (font (size 1.27 1.27)) hide)
     )
@@
   (symbol (lib_id "Device:R_Small") (at 81.28 148.59 180) (unit 1)
     (in_bom yes) (on_board yes) (fields_autoplaced)
-    (property "Reference" "R11" (id 0) (at 78.74 147.3199 0)
+    (property "Reference" "R15" (id 0) (at 78.74 147.3199 0)
       (effects (font (size 1.27 1.27)) (justify left))
     )
@@
       (effects (font (size 1.27 1.27)) hide)
     )
-    (property "LCSC Part Number" "C1711" (id 5) (at 81.28 158.75 0)
+    (property "LCSC Part Number" "C49678" (id 5) (at 81.28 158.75 0)
       (effects (font (size 1.27 1.27)) hide)
     )
@@
   (symbol (lib_id "Device:R_Small") (at 81.28 115.57 180) (unit 1)
     (in_bom yes) (on_board yes) (fields_autoplaced)
-    (property "Reference" "R10" (id 0) (at 78.74 114.2999 0)
-      (effects (font (size 1.27 1.27)) (justify left))
-    )
+    (property "Reference" "R14" (id 0) (at 78.74 114.2999 0)
+      (effects (font (size 1.27 1.27)) (justify left))
+    )
