File: Heatplate_v1.0/Heatplate_v1.0.kicad_pcb (KiCad board)
At the start: 2 copper layers, 100 x 100 mm, 57 parts, among them J1 Barrel_Jack_Switch, Q1 WSP4409A, Q2 IRLR8726TRPBF, Q3 SS8050, SW1 SW_Push, SW2 SW_Push, U1 ATMEGA4809-AFR, U2 AMS1117-5.0

Commit message: Add files via upload
Other:
- board text added: "github.com/DerSpatz/PCB-reflow-solder-heat-plate development by: Bastian Mohing (hardware) Nathan Heidt (software) Merlin Shaw (testing)"
- board text removed: "github.com/DerSpatz/PCB-reflow-solder-heat-plate development by: Bastian Mohing (hardware) Nathan Heidt(software) Merlin Shaw (testing)"
Changed lines of the file:
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@@
   (gr_arc (start 97.65 78.75) (mid 99.9 81) (end 97.65 83.25) (layer "Edge.Cuts") (width 0.05))
   (gr_line (start 160 63.5) (end 160 156.5) (layer "Edge.Cuts") (width 0.05))
-  (gr_text "github.com/DerSpatz/PCB-reflow-solder-heat-plate\ndevelopment by:\nBastian Mohing (hardware)\nNathan Heidt(software)\nMerlin Shaw (testing)" (at 150 93) (layer "B.SilkS")
+  (gr_text "github.com/DerSpatz/PCB-reflow-solder-heat-plate\ndevelopment by:\nBastian Mohing (hardware)\nNathan Heidt (software)\nMerlin Shaw (testing)" (at 150 93) (layer "B.SilkS")
     (effects (font (size 2 1.8) (thickness 0.25)) (justify left mirror))
   )

Commit message: added "JLCJLCJLCJLC"
Other:
- board text added: "JLCJLCJLCJLC"
Changed lines of the file:
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@@
     (effects (font (size 1.4 1.4) (thickness 0.24)) (justify left))
+  )
+  (gr_text "JLCJLCJLCJLC" (at 71.7 64.2) (layer "F.SilkS")
+    (effects (font (size 0.85 0.85) (thickness 0.15)))
   )
   (gr_text "84mm x 70mm" (at 156.25 147.5 90) (layer "F.SilkS")
