File: Heatplate_v1.1/Heatplate_v1.1.kicad_sch (KiCad schematic)
At the start: 45 parts, among them J1 Barrel_Jack_Switch, Q1 WSP4409A, Q2 IRLR8726TRPBF, Q3 SS8050, U1 ATMEGA4809-AFR, U2 AMS1117-5.0

Commit message: minor change to BOM
Parts:
- H1, H2, H3, H4: Information buy M3 studs with 12-15mm length elsewhere -> buy both parts for studs and screws; LCSC Part Number (none) -> C551332; LCSC Part Number Alternative (none) -> C357543
Changed lines of the file:
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@@
       (effects (font (size 1.27 1.27)) hide)
     )
-    (property "Information" "buy M3 studs with 12-15mm length elsewhere" (id 4) (at 44.45 189.23 0)
+    (property "Information" "buy both parts for studs and screws" (id 4) (at 44.45 189.23 0)
+      (effects (font (size 1.27 1.27)) hide)
+    )
+    (property "LCSC Part Number" "C551332" (id 5) (at 44.45 189.23 0)
+      (effects (font (size 1.27 1.27)) hide)
+    )
+    (property "LCSC Part Number Alternative" "C357543" (id 6) (at 44.45 189.23 0)
       (effects (font (size 1.27 1.27)) hide)
     )
@@
       (effects (font (size 1.27 1.27)) hide)
     )
-    (property "Information" "buy M3 studs with 12-15mm length elsewhere" (id 4) (at 25.4 181.61 0)
+    (property "Information" "buy both parts for studs and screws" (id 4) (at 25.4 181.61 0)
+      (effects (font (size 1.27 1.27)) hide)
+    )
+    (property "LCSC Part Number" "C551332" (id 5) (at 25.4 181.61 0)
+      (effects (font (size 1.27 1.27)) hide)
+    )
+    (property "LCSC Part Number Alternative" "C357543" (id 6) (at 25.4 181.61 0)
       (effects (font (size 1.27 1.27)) hide)
     )
@@
       (effects (font (size 1.27 1.27)) hide)
     )
-    (property "Information" "buy M3 studs with 12-15mm length elsewhere" (id 4) (at 44.45 181.61 0)
+    (property "Information" "buy both parts for studs and screws" (id 4) (at 44.45 181.61 0)
+      (effects (font (size 1.27 1.27)) hide)
+    )
+    (property "LCSC Part Number" "C551332" (id 5) (at 44.45 181.61 0)
+      (effects (font (size 1.27 1.27)) hide)
+    )
+    (property "LCSC Part Number Alternative" "C357543" (id 6) (at 44.45 181.61 0)
       (effects (font (size 1.27 1.27)) hide)
     )
@@
       (effects (font (size 1.27 1.27)) hide)
     )
-    (property "Information" "buy M3 studs with 12-15mm length elsewhere" (id 4) (at 25.4 189.23 0)
-      (effects (font (size 1.27 1.27)) hide)
-    )
+    (property "Information" "buy both parts for studs and screws" (id 4) (at 25.4 189.23 0)
+      (effects (font (size 1.27 1.27)) hide)
+    )
+    (property "LCSC Part Number" "C551332" (id 5) (at 25.4 189.23 0)
+      (effects (font (size 1.27 1.27)) hide)
+    )
+    (property "LCSC Part Number Alternative" "C357543" (id 6) (at 25.4 189.23 0)
+      (effects (font (size 1.27 1.27)) hide)
+    )

Commit message: changed R4 from 1k to 4k7
The current flow through this resistor was too high, so it got too hot.
Parts:
- R4: value 1k -> 4k7; Information 1% -> (none); LCSC Part Number C17513 -> C17673; LCSC Part Number Alternative C95781 -> C105427
Changed lines of the file:
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@@
+    (pin "2")
+  )
+  (symbol (lib_id "Device:R_Small") (at 142.24 118.11 180) (unit 1)
+    (in_bom yes) (on_board yes) (fields_autoplaced)
+    (property "Reference" "R4" (id 0) (at 144.78 116.8399 0)
+      (effects (font (size 1.27 1.27)) (justify right))
+    )
+    (property "Value" "4k7" (id 1) (at 144.78 119.3799 0)
+      (effects (font (size 1.27 1.27)) (justify right))
+    )
+    (property "Footprint" "Resistor_SMD:R_0805_2012Metric" (id 2) (at 142.24 118.11 0)
+      (effects (font (size 1.27 1.27)) hide)
+    )
+    (property "Datasheet" "~" (id 3) (at 142.24 118.11 0)
+      (effects (font (size 1.27 1.27)) hide)
+    )
+    (property "LCSC Part Number" "C17673" (id 4) (at 142.24 118.11 0)
+      (effects (font (size 1.27 1.27)) hide)
+    )
+    (property "LCSC Part Number Alternative" "C105427" (id 5) (at 142.24 118.11 0)
+      (effects (font (size 1.27 1.27)) hide)
+    )
+    (pin "1")
     (pin "2")
   )
@@
     (pin "2")
     (pin "3")
-  )
-  (symbol (lib_id "Device:R_Small") (at 142.24 118.11 180) (unit 1)
-    (in_bom yes) (on_board yes) (fields_autoplaced)
-    (property "Reference" "R4" (id 0) (at 144.78 116.8399 0)
-      (effects (font (size 1.27 1.27)) (justify right))
-    )
-    (property "Value" "1k" (id 1) (at 144.78 119.3799 0)
-      (effects (font (size 1.27 1.27)) (justify right))
-    )
-    (property "Footprint" "Resistor_SMD:R_0805_2012Metric" (id 2) (at 142.24 118.11 0)
-      (effects (font (size 1.27 1.27)) hide)
-    )
-    (property "Datasheet" "~" (id 3) (at 142.24 118.11 0)
-      (effects (font (size 1.27 1.27)) hide)
-    )
-    (property "Information" "1%" (id 4) (at 142.24 118.11 0)
-      (effects (font (size 1.27 1.27)) hide)
-    )
-    (property "LCSC Part Number" "C17513" (id 5) (at 142.24 118.11 0)
-      (effects (font (size 1.27 1.27)) hide)
-    )
-    (property "LCSC Part Number Alternative" "C95781" (id 6) (at 142.24 118.11 0)
-      (effects (font (size 1.27 1.27)) hide)
-    )
-    (pin "1")
-    (pin "2")
   )
   (symbol (lib_id "Device:R_Small") (at 26.67 102.87 90) (unit 1)
@@
       (reference "R3") (unit 1) (value "1k") (footprint "Resistor_SMD:R_0805_2012Metric")
     )
-    (path "/c0f3f890-1533-47a0-80d5-bda678f891d3"
-      (reference "R4") (unit 1) (value "1k") (footprint "Resistor_SMD:R_0805_2012Metric")
+    (path "/485fd4d0-7649-4a0a-88ca-2ad442e8583d"
+      (reference "R4") (unit 1) (value "4k7") (footprint "Resistor_SMD:R_0805_2012Metric")
     )
     (path "/42d415a7-d95b-4060-b417-e14fc9a8775b"

Commit message: Add files via upload
Parts:
- Q1: symbol User:Q_NMOS_SSSGDDDD -> User:Q_PMOS_SSSGDDDD
Changed lines of the file:
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@@
     (pin "4")
   )
-  (symbol (lib_id "User:Q_NMOS_SSSGDDDD") (at 63.5 39.37 90) (unit 1)
+  (symbol (lib_id "User:Q_PMOS_SSSGDDDD") (at 63.5 39.37 90) (unit 1)
     (in_bom yes) (on_board yes) (fields_autoplaced)
     (property "Reference" "Q1" (id 0) (at 63.5 29.21 90))
